File: motorgo_core/H_brdige_AP30H80Q.kicad_sch (KiCad schematic)
At the start: 33 parts, among them J8 DNP, Q10 AP30H80Q, Q11 AP30H80Q, Q12 AP30H80Q, Q7 AP30H80Q, Q8 AP30H80Q, Q9 AP30H80Q, U4 FD6288

Commit message: update to recent production
Parts:
- C33: value 100nF -> 100nF 25v
- C34, C39, C46: value 100nF -> 100nF 10v
- D10, D8, D9: value D_Schottky -> D_Schottky C7420331
- J8: now not fitted
Changed lines of the file:
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@@
 		(in_bom yes)
 		(on_board yes)
-		(dnp no)
+		(dnp yes)
 		(property "Reference" "J8"
 			(at 227.0731 116.814 0)
@@
 			)
 		)
-		(property "Value" "100nF"
+		(property "Value" "100nF 10v"
 			(at 187.96 105.41 0)
 			(effects
@@
 			)
 		)
-		(property "Value" "100nF"
+		(property "Value" "100nF 25v"
 			(at 68.58 95.25 0)
 			(effects
@@
 			)
 		)
-		(property "Value" "D_Schottky"
+		(property "Value" "D_Schottky C7420331"
 			(at 163.83 91.1225 90)
 			(effects
@@
 			)
 		)
-		(property "Value" "100nF"
+		(property "Value" "100nF 10v"
 			(at 168.91 95.25 0)
 			(effects
@@
 			)
 		)
-		(property "Value" "100nF"
+		(property "Value" "100nF 10v"
 			(at 147.32 85.09 0)
 			(effects
@@
 			)
 		)
-		(property "Value" "D_Schottky"
+		(property "Value" "D_Schottky C7420331"
 			(at 142.24 80.9625 90)
 			(effects
@@
 			)
 		)
-		(property "Value" "D_Schottky"
+		(property "Value" "D_Schottky C7420331"
 			(at 182.88 101.2825 90)
 			(effects
