File: motorgo_core/LISM6.kicad_sch (KiCad schematic)
At the start: 10 parts, among them U10 LIS3MDLTR, U11 LSM6DS3TR

Commit message: update to recent production
Parts:
- C30, C31: value 100nF -> 100nF 10v
- C32: value 1uF -> 1uF 10v
Changed lines of the file:
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@@
 			)
 		)
-		(property "Value" "100nF"
+		(property "Value" "100nF 10v"
 			(at 64.4602 120.678 0)
 			(effects
@@
 			)
 		)
-		(property "Value" "100nF"
+		(property "Value" "100nF 10v"
 			(at 72.7152 119.987 0)
 			(effects
@@
 			)
 		)
-		(property "Value" "1uF"
+		(property "Value" "1uF 10v"
 			(at 85.09 120.1038 0)
 			(effects
