File: motorgo_core/motor_go_power_system.kicad_sch (KiCad schematic)
At the start: 23 parts, among them U6 TPS54620RHLR, U8 AMS1117-3.3

Commit message: update to recent production
Parts:
- C1: value 68pf -> 68pf 10v
- C15, C2: value 4.7uF 1mOhm -> 4.7uF 1mOhm 25v
- C20: value 6.8nf -> 6.8nf 10v
- C23: value 47uF 3mOhm -> 47uF 3mOhm 25v
- J11: value ~ -> CONN-TH_XT30PW-M
- L1: value 2.2uH 12.7mOhm -> 2.2uH 12.7mOhm C5440776
Other:
- note removed: "CMU requests barrel jack"
Changed lines of the file:
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@@
-		)
-	)
-	(text "CMU requests barrel jack"
-		(exclude_from_sim no)
-		(at 185.42 91.44 0)
-		(effects
-			(font
-				(size 1.27 1.27)
-			)
-			(justify left bottom)
 		)
 	)
@@
 			)
 		)
-		(property "Value" "47uF 3mOhm"
+		(property "Value" "47uF 3mOhm 25v"
 			(at 158.75 80.01 0)
 			(effects
@@
 			)
 		)
-		(property "Value" "~"
+		(property "Value" "CONN-TH_XT30PW-M"
 			(at 197.485 106.045 0)
 			(effects
@@
 			)
 		)
-		(property "Value" "4.7uF 1mOhm"
+		(property "Value" "4.7uF 1mOhm 25v"
 			(at 38.354 77.216 0)
 			(effects
@@
 			)
 		)
-		(property "Value" "6.8nf"
+		(property "Value" "6.8nf 10v"
 			(at 81.407 107.569 0)
 			(effects
@@
 		)
 		(property "Value" "470uF 35V"
-			(at 209.55 109.728 90)
+			(at 211.328 109.474 90)
 			(effects
 				(font
@@
 			)
 		)
-		(property "Value" "68pf"
+		(property "Value" "68pf 10v"
 			(at 97.155 105.41 0)
 			(effects
@@
 			)
 		)
-		(property "Value" "2.2uH 12.7mOhm"
+		(property "Value" "2.2uH 12.7mOhm C5440776"
 			(at 141.605 62.865 90)
 			(effects
@@
 			)
 		)
-		(property "Value" "4.7uF 1mOhm"
+		(property "Value" "4.7uF 1mOhm 25v"
 			(at 38.354 75.184 0)
 			(effects
