File: motorgo_core/motorgo_core.kicad_sch (KiCad schematic)
At the start: 21 parts, among them J1 USB4520-03-0-A_REVA, J12 Conn_01x04_Pin, J4 Conn_02x20_Odd_Even, J5 Conn_01x04_Pin, J9 Conn_01x04_Pin, U1 ESP32-S3-WROOM-1, U2 USBLC6-2P6

Commit message: update to recent production
Parts:
- D1: value LED -> LED blue
- D2: value LED -> LED green
- D3: value LED -> LED red
- J12, J5, J9: now not fitted
- J2, J3: value ~ -> C2886897
Changed lines of the file:
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@@
 		(in_bom yes)
 		(on_board yes)
-		(dnp no)
+		(dnp yes)
 		(property "Reference" "J5"
 			(at 171.958 70.612 0)
@@
 			)
 		)
-		(property "Value" "LED"
+		(property "Value" "LED red"
 			(at 46.99 168.5925 90)
 			(effects
@@
 			)
 		)
-		(property "Value" "LED"
+		(property "Value" "LED blue"
 			(at 27.94 168.5925 90)
 			(effects
@@
 		(in_bom yes)
 		(on_board yes)
-		(dnp no)
+		(dnp yes)
 		(property "Reference" "J9"
 			(at 179.832 70.612 0)
@@
 			)
 		)
-		(property "Value" "LED"
+		(property "Value" "LED green"
 			(at 38.1 168.5925 90)
 			(effects
@@
 			)
 		)
-		(property "Value" "~"
+		(property "Value" "C2886897"
 			(at 167.64 40.005 0)
 			(effects
@@
 		(in_bom yes)
 		(on_board yes)
-		(dnp no)
+		(dnp yes)
 		(property "Reference" "J12"
 			(at 187.452 70.612 0)
@@
 			)
 		)
-		(property "Value" "~"
+		(property "Value" "C2886897"
 			(at 183.515 40.005 0)
 			(effects
